File: Hypnowheel.sch (KiCad schematic (older format))
At the start: 1 part

Commit message: updated LED and TLC5917 symbols; added LEDs to schematic
Parts:
- removed IC?: ATMEGA328-P, DIL28, symbol ATMEGA328-P
- added RGB_LED? (x8): CLV1A-FKB, symbol CLV1A-FKB
- added TLC5917_? (x3): TLC5917IN, symbol TLC5917IN
Connections:
- wire segments 0 -> 66
Changed lines of the file:
@@
-EESchema Schematic File Version 2  date Mon 14 Apr 2014 01:45:21 AM EDT
+EESchema Schematic File Version 2  date Tue 15 Apr 2014 12:24:12 AM EDT
 LIBS:power
 LIBS:device
@@
 LIBS:contrib
 LIBS:valves
+LIBS:Hypnowheel
 LIBS:Hypnowheel-cache
 EELAYER 25  0
@@
 Sheet 1 1
 Title ""
-Date "14 apr 2014"
+Date "15 apr 2014"
 Rev ""
 Comp ""
@@
 Comment4 ""
 $EndDescr
-$Comp
-L ATMEGA328-P IC?
-U 1 1 534B6DDF
-P 7650 4000
-F 0 "IC?" H 6950 5250 50  0000 L BNN
-F 1 "ATMEGA328-P" H 7900 2600 50  0000 L BNN
-F 2 "DIL28" H 7050 2650 50  0001 C CNN
-	1    7650 4000
+Wire Wire Line
+	9650 2650 9650 3400
+Wire Wire Line
+	9650 3400 8250 3400
+Wire Wire Line
+	8250 3400 8250 3750
+Wire Wire Line
+	8950 2650 8950 3200
+Wire Wire Line
+	8950 3200 7950 3200
+Wire Wire Line
+	7950 3200 7950 3750
+Wire Wire Line
+	8250 2650 8250 3000
+Wire Wire Line
+	8250 3000 7650 3000
+Wire Wire Line
+	7650 3000 7650 3750
+Wire Wire Line
+	7550 2650 7550 2800
+Wire Wire Line
+	7550 2800 7350 2800
+Wire Wire Line
+	7350 2800 7350 3750
+Wire Wire Line
+	6850 2650 6850 3050
+Wire Wire Line
+	6850 3050 6050 3050
+Wire Wire Line
+	6050 3050 6050 3750
+Wire Wire Line
+	6150 2650 6150 2900
+Wire Wire Line
+	6150 2900 5750 2900
+Wire Wire Line
+	5750 2900 5750 3750
+Wire Wire Line
+	4400 2650 4400 3000
+Wire Wire Line
+	4400 3000 5000 3000
+Wire Wire Line
+	5000 3000 5000 3750
+Wire Wire Line
+	5100 2650 5100 2800
+Wire Wire Line
+	5100 2800 5300 2800
+Wire Wire Line
+	5300 2800 5300 3750
+Wire Wire Line
+	4050 2650 4050 2800
+Wire Wire Line
+	4050 2800 3850 2800
+Wire Wire Line
+	3850 2800 3850 3750
+Wire Wire Line
+	1950 2650 1950 3200
+Wire Wire Line
+	1950 3200 2950 3200
+Wire Wire Line
+	2950 3200 2950 3700
+Wire Wire Line
+	2650 2650 2650 3000
+Wire Wire Line
+	2650 3000 3250 3000
+Wire Wire Line
+	3250 3000 3250 3750
+Wire Wire Line
+	3350 2650 3350 2800
+Wire Wire Line
+	3350 2800 3550 2800
+Wire Wire Line
+	3550 2800 3550 3750
+Wire Wire Line
+	3700 3750 3700 2650
+Wire Wire Line
+	3400 3750 3400 2900
+Wire Wire Line
+	3400 2900 3000 2900
+Wire Wire Line
+	3000 2900 3000 2650
+Wire Wire Line
+	3100 3750 3100 3100
+Wire Wire Line
+	3100 3100 2300 3100
+Wire Wire Line
+	2300 3100 2300 2650
+Wire Wire Line
+	2800 3750 2800 3300
+Wire Wire Line
+	2800 3300 1600 3300
+Wire Wire Line
+	1600 3300 1600 2650
+Wire Wire Line
+	5450 3750 5450 2650
+Wire Wire Line
+	5150 3750 5150 2900
+Wire Wire Line
+	5150 2900 4750 2900
+Wire Wire Line
+	4750 2900 4750 2650
+Wire Wire Line
+	5600 3750 5600 2800
+Wire Wire Line
+	5600 2800 5800 2800
+Wire Wire Line
+	5800 2800 5800 2650
+Wire Wire Line
+	5900 3750 5900 3000
+Wire Wire Line
+	5900 3000 6500 3000
+Wire Wire Line
+	6500 3000 6500 2650
+Wire Wire Line
+	7200 3750 7200 2650
+Wire Wire Line
+	7500 3750 7500 2900
+Wire Wire Line
+	7500 2900 7900 2900
+Wire Wire Line
+	7900 2900 7900 2650
+Wire Wire Line
+	7800 3750 7800 3100
+Wire Wire Line
+	7800 3100 8600 3100
+Wire Wire Line
+	8600 3100 8600 2650
+Wire Wire Line
+	8100 3750 8100 3300
+Wire Wire Line
+	8100 3300 9300 3300
+Wire Wire Line
+	9300 3300 9300 2650
+$Comp
+L CLV1A-FKB RGB_LED?
+U 1 1 534CB121
+P 9300 1900
+F 0 "RGB_LED?" V 9250 2200 60  0000 C CNN
+F 1 "CLV1A-FKB" V 9250 1600 60  0001 C CNN
+	1    9300 1900
+	0    1    1    0
+$EndComp
+$Comp
+L CLV1A-FKB RGB_LED?
+U 1 1 534CB063
+P 8250 1900
+F 0 "RGB_LED?" V 8200 2200 60  0000 C CNN
+F 1 "CLV1A-FKB" V 8200 1600 60  0001 C CNN
+	1    8250 1900
+	0    1    1    0
+$EndComp
+$Comp
+L CLV1A-FKB RGB_LED?
+U 1 1 534CB061
+P 7200 1900
+F 0 "RGB_LED?" V 7150 2200 60  0000 C CNN
+F 1 "CLV1A-FKB" V 7150 1600 60  0001 C CNN
+	1    7200 1900
+	0    1    1    0
+$EndComp
+$Comp
+L CLV1A-FKB RGB_LED?
+U 1 1 534CB05B
+P 6150 1900
+F 0 "RGB_LED?" V 6100 2200 60  0000 C CNN
+F 1 "CLV1A-FKB" V 6100 1600 60  0001 C CNN
+	1    6150 1900
+	0    1    1    0
+$EndComp
+$Comp
+L CLV1A-FKB RGB_LED?
+U 1 1 534CB058
+P 5100 1900
+F 0 "RGB_LED?" V 5050 2200 60  0000 C CNN
+F 1 "CLV1A-FKB" V 5050 1600 60  0001 C CNN
+	1    5100 1900
+	0    1    1    0
+$EndComp
+$Comp
+L CLV1A-FKB RGB_LED?
+U 1 1 534CB055
+P 4050 1900
+F 0 "RGB_LED?" V 4000 2200 60  0000 C CNN
+F 1 "CLV1A-FKB" V 4000 1600 60  0001 C CNN
+	1    4050 1900
+	0    1    1    0
+$EndComp
+$Comp
+L CLV1A-FKB RGB_LED?
+U 1 1 534CB038
+P 3000 1900
+F 0 "RGB_LED?" V 2950 2200 60  0000 C CNN
+F 1 "CLV1A-FKB" V 2950 1600 60  0001 C CNN
+	1    3000 1900
+	0    1    1    0
+$EndComp
+$Comp
+L TLC5917IN TLC5917_?
+U 1 1 534CAF04
+P 7750 4500
+F 0 "TLC5917_?" V 8500 4200 60  0000 C CNN
+F 1 "TLC5917IN" H 7750 4500 60  0001 C CNN
+	1    7750 4500
 	1    0    0    -1
 $EndComp
+$Comp
+L TLC5917IN TLC5917_?
+U 1 1 534CAE7D
+P 5550 4500
+F 0 "TLC5917_?" V 6300 4200 60  0000 C CNN
+F 1 "TLC5917IN" H 5550 4500 60  0001 C CNN
+	1    5550 4500
+	1    0    0    -1
+$EndComp
+$Comp
+L TLC5917IN TLC5917_?
+U 1 1 534CAE74
+P 3350 4500
+F 0 "TLC5917_?" V 4100 4200 60  0000 C CNN
+F 1 "TLC5917IN" H 3350 4500 60  0001 C CNN
+	1    3350 4500
+	1    0    0    -1
+$EndComp
+$Comp
+L CLV1A-FKB RGB_LED?
+U 1 1 534CA8CC
+P 1950 1900
+F 0 "RGB_LED?" V 1900 2200 60  0000 C CNN
+F 1 "CLV1A-FKB" V 1900 1600 60  0001 C CNN
+	1    1950 1900
+	0    1    1    0
+$EndComp
 $EndSCHEMATC

Commit message: connected LED drivers to each other
Parts:
- added C?: CP1, symbol CP1
- added C? (x3): C, symbol C
- added R? (x3): R, symbol R
Connections:
- net labels added: +5V, CLOCK, DATA_OUT, GND, LATCH
- wire segments 66 -> 106

Commit message: redesigned schematic; driver sheet nearly complete
Parts:
- removed C?: CP1, symbol CP1
- removed C? (x3): C, symbol C
- removed R? (x3): R, symbol R
- removed RGB_LED? (x8): CLV1A-FKB, symbol CLV1A-FKB
- removed TLC5917_? (x3): TLC5917IN, symbol TLC5917IN
Connections:
- net labels removed: +5V, CLOCK, DATA_OUT, GND, LATCH
- wire segments 106 -> 0
